File: Hardware/Spectra1.sch (EAGLE design)
At the start: 43 parts, among them IC2 L293D, IC3 MCP601OT, J2 POWER_JACK, Q1 8/16/20MHz, U2 MCP73831, U3 MIC5205, U4 ATMEGA328

Commit message: Added Updated PCB Specta
Parts:
- removed AMT103-V: PURDUE-EWH-ENCODER, Purdue-EWH-Encoder:PURDUE-EWH-ENCODER
- removed C8, C9: 4.7uF, SparkFun:CAP0402-CAP
- removed D1: RED, SparkFun:LED0603
- removed IC2: L293D, st-microelectronics:L293D
- removed IC3: MCP601OT, CalvEngIO-AnalogIC:MCP601OT
- removed J2: POWER_JACK, SparkFun-Connectors:POWER_JACK
- removed U$1: EWH_KEYPAD, Purdue-EWH-Keypad:EWH_KEYPAD
- added C3, C4: 4.7uF, SparkFun:CAP0402-CAP
- added D11: RED, SparkFun:LED0603
- added IC1: L293D, st-microelectronics:L293D
- added J1: POWER_JACK, SparkFun-Connectors:POWER_JACK
- added JP13, JP5, JP8, JP9: (no value), SparkFun:M02PTH
- added JP3, JP6: M12PTH, SparkFun:M12PTH
- added JP4: (no value), SparkFun:M03PTH
- added JP7: LiPo Battery, SparkFun:M02-JST-2MM-SMT
- added U1: MCP73831, SparkFun:MCP73831
- C1: value (none) -> 1uF; device resistor:C-EUC0603 -> SparkFun:CAP0402-CAP
- C2: value (none) -> 10nF; device resistor:C-EUC0402 -> SparkFun:CAP0402-CAP
- JP1: value LiPo Battery -> input
- JP2: device SparkFun:M02PTH -> SparkFun:M03PTH
- R1: value 10k -> 1k; device SparkFun-Resistors:10KOHM-0603-1/10W-1% -> SparkFun:RESISTOR0402-RES
- R2: value 10k -> 180; device SparkFun-Resistors:10KOHM-0603-1/10W-1% -> SparkFun:RESISTOR0402-RES
- R3: value (none) -> 330; device resistor:R-US_R0402 -> SparkFun:RESISTOR0402-RES
- R4: value (none) -> 2K; device resistor:R-US_R0402 -> SparkFun:RESISTOR0402-RES
- R5, R6: value 10k -> 4.7k; device SparkFun-Resistors:10KOHM-0603-1/10W-1% -> SparkFun:RESISTOR0402-RES
- R7: value 330 -> 4.7k
- R8: value 2K -> 4.7k
- U2: value MCP73831 -> MAX1704X; device SparkFun:MCP73831 -> SparkFun:MAX1704X
Connections:
- removed net 5V: IC2.3-4EN, IC3.V+, R3.2
- removed net D11: AMT103-V.B, U4.PB3(MOSI/OC2)
- removed net N$12: U$1.D7
- removed net N$13: R2.2, U$1.D6
- removed net N$14: R6.2, U$1.D4
- removed net N$16: R5.2, U$1.D5
- removed net N$17: D1.A, R7.1
- removed net N$18: IC3.-IN, IC3.OUT
- removed net N$8: C2.1, IC2.VCC1
- removed net PROG1: R8.1, U2.PROG
- removed net STAT1: D1.C, U2.STAT
- removed net STEPPER_ROB-10846: IC2.1Y, IC2.2Y, IC2.3Y, IC2.4Y
- new net ALT: JP4.3, R5.1, U2.ALT
- new net D7: JP3.3
- new net MISO: JP6.10, U4.PB4(MISO)
- new net MOSI: JP6.11, U4.PB3(MOSI/OC2)
- new net PROG: R4.1, U1.PROG
- new net QST: JP2.3, R6.2, U2.QST
- new net SCL: JP2.2, R7.1, U2.SCL
- new net SDA: JP2.1, R8.1, U2.SDA
- new net STAT: D11.C, U1.STAT
- new net VDD: C2.1, R2.1, U2.VDD
- net A0: now also JP6.8; no longer IC2.1A
- net A1: now also JP6.7; no longer IC2.2A
- net A2: now also JP6.6; no longer IC2.4A
- net A3: now also JP6.5; no longer IC2.3A
- net A4: now also JP9.1
- net A5: now also JP9.2
- net A6: now also JP13.1
- net A7: now also JP13.2
- net CHRG.CTRL: now also R4.2, U4.PD7(AIN1); no longer R8.2, U4.PB4(MISO)
- net D10: now also JP6.12; no longer U$1.D10
- net D2: now also JP3.8
- net D3: now also JP3.7
- net D4: now also JP3.6
- net D5: now also JP3.5
- net D6: now also JP3.4
- net D8: now also JP3.2; no longer R1.2, U$1.D8
- net D9: now also JP3.1; no longer U$1.D9
- net GND: now also C2.2, C3.2, C4.2, JP3.9, JP4.2, JP5.2, JP6.2, JP7.1, JP8.1, R6.1, U1.VSS, U2.CTG, U2.GND@4, U2.GND@EP; no longer AMT103-V.SW-, C8.2, C9.2, IC2.GND1, IC2.GND2, IC2.GND3, IC2.GND4, IC3.V-, J2.GND, J2.GNDBREAK, JP2.1, R4.1, U2.VSS
- net N$2: now also R1.2, U2.CELL; no longer IC2.VCC2
- net N$3: now also D11.A; no longer IC3.+IN, R4.2
- net RAW: now also JP6.1
- net RESET: now also JP3.10, JP6.3
- net RXI: now also JP3.11
- net SCK: now also JP6.9
- net TXO: now also JP3.12
- net VCC: now also C4.1, JP4.1, JP5.1, JP6.4, JP7.2, JP8.2, R2.2, R5.2, R7.2, R8.2, U1.VBAT; no longer AMT103-V.SW+, C9.1, IC2.1-2EN, JP2.2, R2.1, R5.1, R6.1, U2.VBAT
- net VIN: now also C3.1, R3.2, U1.VIN; no longer C8.1, J2.PWR, R7.2, U2.VIN
Other:
- note added: "Off Grid Breakout headers"
- note removed: "#"
- note removed: "*"
- note removed: "0"
- note removed: "1"
- note removed: "2"
- note removed: "3"
- note removed: "4"
- note removed: "5"
- note removed: "6"
- note removed: "7"
- note removed: "8"
- note removed: "9"
- note removed: "<KEYPAD COM-08653"
- moved on the sheet: C1, C10, C13, C19, C2, JP1, LED1, R11, R3, R4, R7, R8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
