File: Hardware/SpectraPCB-V3.brd (EAGLE design)
At the start: 172.7 x 602.9 mm, 36 parts, among them IC1 L293D, IC2 MCP601OT, J1 POWER_JACK, J2 AVR_SPI_PROG_3X2NS, U1 MCP73831

Commit message: Updated SpectaPCB-V3
Parts:
- removed BOOT, BT: (no value), SparkFun-Connectors:1X04_NO_SILK
- removed D2: (no value), CalvEngIO-LED:LED-0603
- removed FTDI: (no value), SparkFun-Connectors:1X05_NO_SILK
- removed R21: 10k, CalvEngIO-Passives:R0402
- added C9: 0.1uF, SparkFun-Capacitors:0603
- added R10: 470, SparkFun-Resistors:0603
- added U$5: LCD-16X2-SERIAL, Purdue-EWH-Displays:LCD-16X2-SERIAL
- added U$6: TSL235R, Purdue-EWH-Sensors:TSL235R
- moved C6 666.8 mm to (14.0, 62.2)
- moved RESET 660.1 mm to (44.5, 44.5)
- moved C8 657.7 mm to (39.4, 52.1)
- moved R9 656.6 mm to (33.0, 52.1)
- moved C5 651.6 mm to (26.7, 47.0), turned to 180 degrees
- moved U$7 649.7 mm to (24.1, 43.2)
- moved C7 645.2 mm to (21.6, 40.6)
- moved ARDUINO 631.3 mm to (33.0, 41.9)
- moved J2 587.7 mm to (50.8, 52.1)
- moved D1 570.4 mm to (76.2, 52.1)
- moved R7 559.3 mm to (60.9, 59.8)
- moved R8 559.3 mm to (66.6, 66.6)
- moved IC2 559.2 mm to (55.9, 66.0)
- moved JP8 524.6 mm to (40.0, 77.9)
- moved JP7 523.3 mm to (49.6, 75.0)
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Connections:
- net LD15 renamed A7
- net LD16 renamed A6
- net N$9 renamed VDD
- net SW5 renamed A4
- net SW6 renamed A5
- removed net 3.3V: BT.1, FTDI.2
- removed net BT-RX: BT.4
- removed net BT-TX: BT.3
- removed net D11-MOSI: BOOT.3
- removed net D12-MISO: BOOT.2
- removed net D13-SCK: BOOT.1
- removed net LD1: ARDUINO.17, R21.1
- removed net LD10: ARDUINO.2
- removed net LD11: ARDUINO.1
- removed net LD12: ARDUINO.32
- removed net LD2: ARDUINO.16
- removed net LD3: ARDUINO.15
- removed net LD4: ARDUINO.14
- removed net LD5: ARDUINO.13
- removed net LD6: ARDUINO.12
- removed net LD7: ARDUINO.11
- removed net LD8: ARDUINO.10
- removed net LD9: ARDUINO.9
- removed net N$10: R3.2, U$1.D5
- removed net N$3: U$1.D10
- removed net N$4: U$1.D9
- removed net N$5: R1.2, U$1.D8/VDD
- removed net N$6: U$1.D7
- removed net N$7: R2.2, U$1.D6
- removed net N$8: R4.2, U$1.D4
- removed net RXI/FTDI/LD13: ARDUINO.31, FTDI.4
- removed net SW1: ARDUINO.23
- removed net SW2: ARDUINO.24
- removed net SW3: ARDUINO.25
- removed net SW4: ARDUINO.26
- removed net TXO/FTDI/LD14: ARDUINO.30, FTDI.3
- new net D0: ARDUINO.30
- new net D1: ARDUINO.31, U$5.RX
- new net D10: ARDUINO.14, U$1.D10
- new net D13: ARDUINO.17, R10.2
- new net D2: ARDUINO.32, U$6.OUT
- new net D4: ARDUINO.2, R4.2, U$1.D4
- new net D5: ARDUINO.9, R3.2, U$1.D5
- new net D6: ARDUINO.10, R2.2, U$1.D6
- new net D7: ARDUINO.11, U$1.D7
- new net D8: ARDUINO.12, R1.2, U$1.D8/VDD
- new net D9: ARDUINO.13, U$1.D9
- net 5V: now also C9.2, U$6.VDD; no longer IC1.1, IC1.9
- net A0: now also ARDUINO.23
- net A1: now also ARDUINO.24
- net A2: now also ARDUINO.25
- net A3: now also ARDUINO.26
- net CHRG.CTRL: now also ARDUINO.16
- net D11: now also ARDUINO.15
- net D3: now also ARDUINO.1
- net DTR: no longer FTDI.5
- net GND: now also C9.1, D1.K, U$5.GND, U$6.GND; no longer BT.2, D2.C, FTDI.1
- net N$16: now also D1.A, R10.1; no longer D2.A, R21.2
- net RESET: no longer BOOT.4
- net VCC: now also IC1.1, IC1.9, U$5.5V
Routing:
- net VCC: track 17.2 -> 89.3 mm
- net D4: track 0.00 -> 69.4 mm
- net D13: track 0.00 -> 36.1 mm
- net N$8: track 26.7 -> 0.00 mm
- net GND: track 42.9 -> 67.5 mm
- net 5V: track 32.1 -> 9.11 mm
- net D5: track 0.00 -> 14.5 mm
- net N$16: track 0.00 -> 13.1 mm
- net D6: track 0.00 -> 10.1 mm
- net VLIPO: track 0.00 -> 8.62 mm
- net RESET: track 0.00 -> 7.41 mm
- net D8: track 0.00 -> 6.45 mm
- net N$7: track 5.89 -> 0.00 mm
- net N$10: track 5.44 -> 0.00 mm
- net N$5: track 5.41 -> 0.00 mm
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Other:
- board size 172.7 x 602.9 mm -> 172.7 x 581.3 mm

Commit message: Updated SpectaPCB-V3
Parts:
- moved U$7 60.3 mm to (83.8, 34.3), turned to 180 degrees
- moved AMT103-V 57.2 mm to (83.8, 20.3), turned to 270 degrees
- moved R2 56.8 mm to (106.7, 36.8)
- moved R1 56.8 mm to (102.9, 36.8)
- moved R4 56.8 mm to (102.9, 39.4)
- moved R3 56.8 mm to (110.5, 36.8)
- moved U$1 55.9 mm to (97.8, 27.9)
- moved R6 52.6 mm to (87.8, 74.8)
- moved C5 50.4 mm to (74.9, 32.4), turned to 0 degrees
- moved D11 49.9 mm to (82.9, 84.4)
- moved C3 49.9 mm to (80.4, 81.8)
- moved C4 49.9 mm to (83.7, 81.8)
- moved JP8 49.9 mm to (89.5, 84.2)
- moved R5 49.9 mm to (79.7, 84.2)
- moved U1 49.9 mm to (81.6, 79.1)
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Connections:
- net 5V: no longer AMT103-V.SW+, C9.2, U$6.VDD
- net VCC: now also AMT103-V.SW+, C9.2, U$6.VDD
Routing:
- net GND: track 67.5 -> 247.8 mm, vias 2 -> 7
- net VCC: track 89.3 -> 174.9 mm, vias 0 -> 4
- net A1: track 0.00 -> 71.9 mm, vias 0 -> 1
- net A0: track 0.00 -> 60.9 mm, vias 0 -> 2
- net D11: track 0.00 -> 51.5 mm, vias 0 -> 1
- net RESET: track 7.41 -> 55.1 mm, vias 0 -> 5
- net D1: track 0.00 -> 47.0 mm, vias 0 -> 1
- net D2: track 0.00 -> 45.1 mm, vias 0 -> 1
- net D3: track 0.00 -> 39.7 mm, vias 0 -> 1
- net VLIPO: track 8.62 -> 48.3 mm, vias 0 -> 2
- net CHRG.CTRL: track 0.00 -> 32.6 mm
- net A2: track 0.00 -> 27.5 mm, vias 0 -> 2
- net D5: track 14.5 -> 41.9 mm
- net A3: track 0.00 -> 27.4 mm, vias 0 -> 1
- net D6: track 10.1 -> 35.7 mm
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- added copper zone on layer 16, net GND
- added copper zone on layer 1, net VCC
Other:
- board size 172.7 x 581.3 mm -> 160 x 106.3 mm
- board text added: "<Control System"
