File: Hardware/SpectraPCB-V3.sch (EAGLE design)
At the start: 36 parts, among them IC1 L293D, IC2 MCP601OT, J1 POWER_JACK, J2 AVR_SPI_PROG_3X2NS, U1 MCP73831

Commit message: Updated SpectaPCB-V3
Parts:
- removed BOOT, BT: (no value), SparkFun-Connectors:M041X04_NO_SILK
- removed D2: (no value), CalvEngIO-LED:LED0603
- removed FTDI: (no value), SparkFun-Connectors:M05NO_SILK
- removed R21: 10k, CalvEngIO-Passives:RESISTOR0402
- added C9: 0.1uF, SparkFun-Capacitors:0.1UF-0603-25V-(+80/-20%)
- added R10: 470, SparkFun-Resistors:470OHM-0603-1/10W-1%
- added U$5: LCD-16X2-SERIAL, Purdue-EWH-Displays:LCD-16X2-SERIAL
- added U$6: TSL235R, Purdue-EWH-Sensors:TSL235R
Connections:
- net LD15 renamed A7
- net LD16 renamed A6
- net N$9 renamed VDD
- net SW5 renamed A4
- net SW6 renamed A5
- removed net 3.3V: BT.1, FTDI.2
- removed net BT-RX: BT.4
- removed net BT-TX: BT.3
- removed net D11-MOSI: BOOT.3
- removed net D12-MISO: BOOT.2
- removed net D13-SCK: BOOT.1
- removed net LD1: ARDUINO.PB5(SCK), R21.1
- removed net LD10: ARDUINO.PD4(XCK/T0)
- removed net LD11: ARDUINO.PD3(INT1)
- removed net LD12: ARDUINO.PD2(INT0)
- removed net LD2: ARDUINO.PB4(MISO)
- removed net LD3: ARDUINO.PB3(MOSI/OC2)
- removed net LD4: ARDUINO.PB2(SS/OC1B)
- removed net LD5: ARDUINO.PB1(OC1A)
- removed net LD6: ARDUINO.PB0(ICP)
- removed net LD7: ARDUINO.PD7(AIN1)
- removed net LD8: ARDUINO.PD6(AIN0)
- removed net LD9: ARDUINO.PD5(T1)
- removed net N$10: R3.2, U$1.D5
- removed net N$3: U$1.D10
- removed net N$4: U$1.D9
- removed net N$5: R1.2, U$1.D8
- removed net N$6: U$1.D7
- removed net N$7: R2.2, U$1.D6
- removed net N$8: R4.2, U$1.D4
- removed net RXI/FTDI/LD13: ARDUINO.PD1(TXD), FTDI.4
- removed net SW1: ARDUINO.PC0(ADC0)
- removed net SW2: ARDUINO.PC1(ADC1)
- removed net SW3: ARDUINO.PC2(ADC2)
- removed net SW4: ARDUINO.PC3(ADC3)
- removed net TXO/FTDI/LD14: ARDUINO.PD0(RXD), FTDI.3
- new net D0: ARDUINO.PD0(RXD)
- new net D1: ARDUINO.PD1(TXD), U$5.RX
- new net D10: ARDUINO.PB2(SS/OC1B), U$1.D10
- new net D13: ARDUINO.PB5(SCK), R10.2
- new net D2: ARDUINO.PD2(INT0), U$6.OUT
- new net D4: ARDUINO.PD4(XCK/T0), R4.2, U$1.D4
- new net D5: ARDUINO.PD5(T1), R3.2, U$1.D5
- new net D6: ARDUINO.PD6(AIN0), R2.2, U$1.D6
- new net D7: ARDUINO.PD7(AIN1), U$1.D7
- new net D8: ARDUINO.PB0(ICP), R1.2, U$1.D8
- new net D9: ARDUINO.PB1(OC1A), U$1.D9
- net 5V: now also C9.2, U$6.VDD; no longer IC1.1-2EN, IC1.3-4EN
- net A0: now also ARDUINO.PC0(ADC0)
- net A1: now also ARDUINO.PC1(ADC1)
- net A2: now also ARDUINO.PC2(ADC2)
- net A3: now also ARDUINO.PC3(ADC3)
- net CHRG.CTRL: now also ARDUINO.PB4(MISO)
- net D11: now also ARDUINO.PB3(MOSI/OC2)
- net D3: now also ARDUINO.PD3(INT1)
- net DTR: no longer FTDI.5
- net GND: now also C9.1, D1.C, U$5.GND, U$6.GND; no longer BT.2, D2.C, FTDI.1
- net N$16: now also D1.A, R10.1; no longer D2.A, R21.2
- net RESET: no longer BOOT.4
- net VCC: now also IC1.1-2EN, IC1.3-4EN, U$5.5V
Other:
- note removed: "Bluetooth"
- note removed: "Bootloading"
- note removed: "FTDI"
- moved on the sheet: D1

Commit message: Updated SpectaPCB-V3
Connections:
- net 5V: no longer AMT103-V.SW+, C9.2, U$6.VDD
- net VCC: now also AMT103-V.SW+, C9.2, U$6.VDD
Other:
- moved on the sheet: AMT103-V, C1, C2, C3, C4, C9, D11, IC1, IC2, J1, JP7, JP8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
